File: Board/UPPSU.sch (KiCad schematic (older format))
At the start: 47 parts, among them J1 Conn_01x04_Male, J2 Conn_01x03, J3 Conn_01x04, J4 ARDUINO, J5 ARDUINO, J6 Conn_02x05_Odd_Even, J7 Conn_01x04_Male, K1 FINDER-30.22, Q1 BC547, U1 AMSRI-7805-NZ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

Commit message: FIX
Connections:
- net +5V: now also J4.9 (Pin_9)
Changed lines of the file:
@@
 	4800 4500 5100 4500
 Wire Wire Line
-	5100 4500 7900 4500
+	5100 4500 7250 4500
 $Comp
 L Connector_Generic:Conn_01x12 J4
@@
 Wire Wire Line
 	5800 5050 5800 4250
+Wire Wire Line
+	6600 6100 6600 6250
+Wire Wire Line
+	6600 6250 7250 6250
+Wire Wire Line
+	7250 6250 7250 4500
+Connection ~ 7250 4500
+Wire Wire Line
+	7250 4500 7900 4500
 $EndSCHEMATC

Commit message: FIX
Parts:
- added J8: Conn_01x04, Connector_PinHeader_2.54mm:PinHeader_1x04_P2.54mm_Vertical, symbol Connector_Generic:Conn_01x04
Connections:
- net at U3.12 (A): now also J7.3 (Pin_3), J8.3 (Pin_3); no longer J7.1 (Pin_1)
- net at J7.2 (Pin_2), U3.13 (B): now also J8.2 (Pin_2)
- net at C9.2, J7.4 (Pin_4), U3.15 (GND2)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: now also J8.4 (Pin_4)
- net at C9.1, U3.16 (VDD2): now also J7.1 (Pin_1), J8.1 (Pin_1); no longer J7.3 (Pin_3)
Other:
- moved on the sheet: J7
Changed lines of the file:
@@
 Wire Wire Line
 	9950 5850 9950 6050
-Connection ~ 9950 6050
 Wire Wire Line
 	9950 5550 9950 4650
-Connection ~ 9950 4650
 $Comp
 L Device:CP C1
@@
 	9700 2200 9800 2200
 Wire Wire Line
-	9950 4650 10300 4650
-Wire Wire Line
-	9950 6050 10300 6050
-Wire Wire Line
 	1100 1950 1100 1850
 Wire Wire Line
@@
 L Connector:Conn_01x04_Male J7
 U 1 1 603AA54F
-P 10900 5250
-F 0 "J7" H 11008 5531 50  0000 C CNN
-F 1 "Conn_01x04_Male" H 11008 5440 50  0000 C CNN
-F 2 "Connector_Phoenix_MSTB:PhoenixContact_MSTBVA_2,5_4-G-5,08_1x04_P5.08mm_Vertical" H 10900 5250 50  0001 C CNN
-F 3 "~" H 10900 5250 50  0001 C CNN
-	1    10900 5250
+P 10500 5150
+F 0 "J7" H 10608 5431 50  0000 C CNN
+F 1 "Conn_01x04_Male" H 10608 5340 50  0000 C CNN
+F 2 "Connector_Phoenix_MSTB:PhoenixContact_MSTBVA_2,5_4-G-5,08_1x04_P5.08mm_Vertical" H 10500 5150 50  0001 C CNN
+F 3 "~" H 10500 5150 50  0001 C CNN
+	1    10500 5150
 	-1   0    0    -1
 $EndComp
-Wire Wire Line
-	10700 5150 9650 5150
-Wire Wire Line
-	10700 5250 9650 5250
-Wire Wire Line
-	9650 5250 9650 5350
-Wire Wire Line
-	10700 5450 10300 5450
-Wire Wire Line
-	10300 5450 10300 6050
-Wire Wire Line
-	10700 5350 10300 5350
-Wire Wire Line
-	10300 5350 10300 4650
 $Comp
 L Connector_Generic:Conn_01x12 J5
@@
 Wire Wire Line
 	7250 4500 7900 4500
+Wire Wire Line
+	9950 6050 10300 6050
+Wire Wire Line
+	10300 6050 10300 5350
+Connection ~ 9950 6050
+Wire Wire Line
+	9950 4650 10300 4650
+Wire Wire Line
+	10300 4650 10300 5050
+Connection ~ 9950 4650
+Wire Wire Line
+	9650 5150 9700 5150
+Wire Wire Line
+	9700 5150 9700 5250
+Wire Wire Line
+	9700 5250 10300 5250
+Wire Wire Line
+	9650 5350 9850 5350
+Wire Wire Line
+	9850 5350 9850 5150
+Wire Wire Line
+	9850 5150 10300 5150
+$Comp
+L Connector_Generic:Conn_01x04 J8
+U 1 1 605FB7AE
+P 10950 5150
+F 0 "J8" V 10822 5330 50  0000 L CNN
+F 1 "Conn_01x04" V 10913 5330 50  0000 L CNN
+F 2 "Connector_PinHeader_2.54mm:PinHeader_1x04_P2.54mm_Vertical" H 10950 5150 50  0001 C CNN
+F 3 "~" H 10950 5150 50  0001 C CNN
+	1    10950 5150
+	1    0    0    -1
+$EndComp
+Wire Wire Line
+	10750 5050 10750 4650
+Wire Wire Line
+	10750 4650 10300 4650
+Connection ~ 10300 4650
+Wire Wire Line
+	10300 6050 10750 6050
+Wire Wire Line
+	10750 6050 10750 5350
+Connection ~ 10300 6050
+Wire Wire Line
+	10750 5150 10300 5150
+Connection ~ 10300 5150
+Wire Wire Line
+	10750 5250 10300 5250
+Connection ~ 10300 5250
 $EndSCHEMATC
