File: Board/UPPSU.kicad_pcb (KiCad board)
At the start: 2 copper layers, 54 parts, among them J1 Conn_01x04_Male, J2 Conn_01x03, J3 Conn_01x04, J4 ARDUINO, J5 ARDUINO, J6 Conn_02x05_Odd_Even, J7 Conn_01x04_Male, K1 FINDER-30.22, Q1 BC547, U1 AMSRI-7805-NZ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

Commit message: Board update
Parts:
- removed the REF** at (149.2, 81.9)
- moved J5 67.0 mm to (156.2, 108.0), turned to 270 degrees
- moved C8 38.1 mm to (175.9, 116.8)
- moved C4 37.9 mm to (132.1, 92.7)
- moved R4 37.9 mm to (146.1, 89.5)
- moved C1 37.9 mm to (109.2, 90.2)
- moved C5 37.9 mm to (125.7, 115.5)
- moved C6 37.9 mm to (152.4, 90.2)
- moved D1 37.9 mm to (125.7, 89.5)
- moved D2 37.9 mm to (174.0, 81.3)
- moved D3 37.9 mm to (196.8, 88.9)
- moved J1 37.9 mm to (105.4, 114.3)
- moved J6 37.9 mm to (200.7, 91.4)
- moved K1 37.9 mm to (176.5, 88.9)
- moved Q1 37.9 mm to (176.5, 95.2)
- moved R1 37.9 mm to (138.4, 89.5)
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Connections:
- J4 pad 9: /+5V -> Net-(J4-Pad9)
- J5 pad 10: Net-(J5-Pad10) -> Net-(J3-Pad1)
- J5 pad 11: Net-(J3-Pad1) -> Net-(J3-Pad3)
- J5 pad 12: Net-(J3-Pad3) -> Net-(J5-Pad12)
- R11 pad 2: Net-(J4-Pad6) -> Net-(J4-Pad7)
- R13 pad 2: Net-(J4-Pad5) -> Net-(J4-Pad8)
- R14 pad 1: Net-(J4-Pad5) -> Net-(J4-Pad8)
- R15 pad 2: Net-(J4-Pad4) -> Net-(J5-Pad5)
- R5 pad 1: Net-(J4-Pad2) -> Net-(J5-Pad12)
- R6 pad 1: Net-(J4-Pad1) -> Net-(J5-Pad6)
- U2 pad 14: Net-(J4-Pad3) -> Net-(J5-Pad9)
- U2 pad 8: Net-(J4-Pad6) -> Net-(J4-Pad7)
- U3 pad 4: Net-(J5-Pad5) -> Net-(J5-Pad8)
- U3 pad 5: Net-(J5-Pad5) -> Net-(J5-Pad8)
- U3 pad 7: Net-(J5-Pad6) -> Net-(J5-Pad7)
Routing:
- net Net-(J5-Pad9): track 0.00 -> 86.8 mm, vias 0 -> 4
- net Net-(J4-Pad3): track 67.7 -> 0.00 mm, vias 2 -> 0
- net Net-(J4-Pad7): track 0.00 -> 61.2 mm, vias 0 -> 2
- net Net-(J4-Pad6): track 47.5 -> 0.00 mm, vias 2 -> 0
- net Net-(J4-Pad8): track 0.00 -> 45.0 mm, vias 0 -> 2
- net Net-(J5-Pad8): track 0.00 -> 44.1 mm, vias 0 -> 2
- net Net-(J5-Pad6): track 54.6 -> 12.9 mm, vias 2 -> 0
- net Net-(J5-Pad7): track 0.00 -> 41.6 mm, vias 0 -> 2
- net Net-(J5-Pad1): track 62.2 -> 23.3 mm
- net Net-(J4-Pad5): track 32.9 -> 0.00 mm, vias 2 -> 0
- net Net-(J5-Pad2): track 59.4 -> 29.1 mm
- net Net-(J3-Pad1): track 35.4 -> 8.94 mm
- net Net-(J4-Pad4): track 26.0 -> 0.00 mm
- net Net-(J5-Pad5): track 54.1 -> 31.1 mm
- net Net-(J4-Pad2): track 21.3 -> 0.00 mm
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Other:
- rule trace_min: 0.2 -> 0.5
- board text added: "Bottom"
- board text added: "VasiKisha"

Commit message: FIX
Connections:
- J4 pad 9: Net-(J4-Pad9) -> /+5V
Routing:
- net /+5V: track 147.1 -> 168.3 mm
- net GND: track 321.4 -> 339.5 mm, vias 4 -> 2
- net Net-(J4-Pad8): track 45.0 -> 44.0 mm

Commit message: FIX
Parts:
- added J8: Conn_01x04, Connector_PinHeader_2.54mm:PinHeader_1x04_P2.54mm_Vertical, F.Cu at (192.4, 114.3)
Connections:
- J7 pad 1: Net-(J7-Pad1) -> Net-(C9-Pad1)
- J7 pad 3: Net-(C9-Pad1) -> Net-(J7-Pad3)
- U3 pad 12: Net-(J7-Pad1) -> Net-(J7-Pad3)
Routing:
- net Net-(J7-Pad1): track 31.0 -> 0.00 mm
- net Net-(J7-Pad3): track 0.00 -> 12.2 mm
- net Net-(J7-Pad2): track 23.4 -> 11.6 mm
- net Net-(C9-Pad1): track 17.9 -> 13.1 mm
- net Net-(C9-Pad2): track 27.6 -> 28.9 mm
Other:
- board text added: "+"
- board text added: "-"
- board text added: "A"
- board text added: "B"
